Commit message: update arm init pose

File: assets/robot/atlas_description/urdf/atlas_allegro_right.urdf (robot description, URDF)
Before this commit: robot multisense_sl, 53 links, 52 joints
Joints:
- joint l_arm_shz: limit lower=-1.5708 upper=0.785398 effort=87 velocity=12 -> lower=-2 upper=0 effort=87 velocity=12
- joint r_arm_shz: limit lower=-0.785398 upper=1.5708 effort=87 velocity=12 -> lower=0 upper=2 effort=87 velocity=12

Commit message: urdf update

File: assets/robot/atlas_description/urdf/atlas_allegro_right.urdf (robot description, URDF)
Before this commit: robot multisense_sl, 53 links, 52 joints
Joints:
- joint r_arm_wry2: origin xyz=0 -0.21 0 rpy=1.57 1.57 0 -> xyz=0 -0.21 0 rpy=1.57 0 0

Commit message: laptop tune initial pose

File: assets/robot/atlas_description/urdf/atlas_allegro_right.urdf (robot description, URDF)
Before this commit: robot multisense_sl, 53 links, 52 joints
Joints:
- joint r_arm_wry2: origin xyz=0 -0.21 0 rpy=1.57 0 0 -> xyz=0 -0.21 0 rpy=1.57 -1.57 0

Commit message: test palm handle distance reward
Co-authored-by: Gavin Chen <idlesilver@users.noreply.github.com>

File: assets/robot/atlas_description/urdf/atlas_allegro_right.urdf (robot description, URDF)
Before this commit: robot multisense_sl, 53 links, 52 joints
Links:
- added link l_palm; visual sphere radius=0.02
Joints:
- added joint virtual_hand: type fixed, parent l_hand, child l_palm, origin xyz=0 -0.15 0 rpy=0 -0 0, axis 0 0 1

Commit message: update bucket Rl train

File: assets/robot/atlas_description/urdf/atlas_allegro_right.urdf (robot description, URDF)
Before this commit: robot multisense_sl, 53 links, 52 joints
Links:
- added link l_palm; visual sphere radius=0.02
Joints:
- added joint virtual_hand: type fixed, parent l_hand, child l_palm, origin xyz=0 -0.15 0 rpy=0 -0 0, axis 0 0 1
- joint r_arm_wry2: origin xyz=0 -0.21 0 rpy=1.57 1.57 0 -> xyz=0 -0.21 0 rpy=1.57 -1.57 0
